File: board/board.kicad_pcb (KiCad board)
At the start: 2 copper layers, 21 x 13 mm, 1 part

Commit message: initial
Parts:
- added J1: M12, b160:M12-6A, F.Cu at (154.2, 96.5)
Changed lines of the file:
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@@
 	)
 	(net 0 "")
+	(net 1 "unconnected-(J1-Pad4)")
+	(net 2 "unconnected-(J1-Pad2)")
+	(net 3 "unconnected-(J1-Pad3)")
+	(net 4 "unconnected-(J1-Pad1)")
+	(net 5 "unconnected-(J1-Pad6)")
+	(net 6 "unconnected-(J1-Pad5)")
 	(footprint "Symbol:OSHW-Symbol_6.7x6mm_SilkScreen"
 		(layer "F.Cu")
@@
 			)
 		)
-		(property "Footprint" ""
+		(property "Footprint" "Symbol:OSHW-Symbol_6.7x6mm_SilkScreen"
 			(at 0 0 0)
 			(unlocked yes)
@@
 				(font
 					(size 1.27 1.27)
+					(thickness 0.15)
 				)
 			)
@@
 				(font
 					(size 1.27 1.27)
+					(thickness 0.15)
 				)
 			)
@@
 				(font
 					(size 1.27 1.27)
-				)
-			)
-		)
+					(thickness 0.15)
+				)
+			)
+		)
+		(sheetname "Root")
 		(sheetfile "board.kicad_sch")
 		(attr exclude_from_pos_files)
@@
 		)
 	)
+	(footprint "b160:M12-6A"
+		(layer "F.Cu")
+		(at 154.21 96.55)
+		(property "Reference" "J1"
+			(at 0 -0.5 0)
+			(unlocked yes)
+			(layer "F.SilkS")
+			(effects
+				(font
+					(size 1 1)
+					(thickness 0.1)
+				)
+			)
+		)
+		(property "Value" "M12"
+			(at 0 1 0)
+			(unlocked yes)
+			(layer "F.Fab")
+			(effects
+				(font
+					(size 1 1)
+					(thickness 0.15)
+				)
+			)
+		)
+		(property "Footprint" "b160:M12-6A"
+			(at 0 0 0)
+			(unlocked yes)
+			(layer "F.Fab")
+			(hide yes)
+			(effects
+				(font
+					(size 1 1)
+					(thickness 0.15)
+				)
+			)
+		)
+		(property "Datasheet" ""
+			(at 0 0 0)
+			(unlocked yes)
+			(layer "F.Fab")
+			(hide yes)
+			(effects
+				(font
+					(size 1 1)
+					(thickness 0.15)
+				)
+			)
+		)
+		(property "Description" ""
+			(at 0 0 0)
+			(unlocked yes)
+			(layer "F.Fab")
+			(hide yes)
+			(effects
+				(font
+					(size 1 1)
+					(thickness 0.15)
+				)
+			)
+		)
+		(property ki_fp_filters "DIN*")
+		(sheetname "Root")
+		(sheetfile "board.kicad_sch")
+		(attr through_hole)
+		(fp_circle
+			(center 0 0)
+			(end 0 -2.25)
+			(stroke
+				(width 0.1)
+				(type default)
+			)
+			(fill none)
+			(layer "Dwgs.User")
+		)
+		(fp_circle
+			(center 0 0)
+			(end 0 -3.95)
+			(stroke
+				(width 0.05)
+				(type default)
+			)
+			(fill none)
+			(layer "F.CrtYd")
+		)
+		(fp_text user "${REFERENCE}"
+			(at 0 2.5 0)
+			(unlocked yes)
+			(layer "F.Fab")
+			(effects
+				(font
+					(size 1 1)
+					(thickness 0.15)
+				)
+			)
+		)
+		(pad "1" thru_hole circle
+			(at -1.25 -1.9)
+			(size 1.75 1.75)
+			(drill 1)
+			(layers "*.Cu" "*.Mask")
+			(remove_unused_layers no)
+			(net 4 "unconnected-(J1-Pad1)")
+			(pintype "passive")
+		)
+		(pad "2" thru_hole circle
+			(at 1.2 -1.9)
+			(size 1.75 1.75)
+			(drill 1)
+			(layers "*.Cu" "*.Mask")
+			(remove_unused_layers no)
+			(net 2 "unconnected-(J1-Pad2)")
+			(pintype "passive")
+		)
+		(pad "3" thru_hole circle
+			(at 2.2 -0.3)
+			(size 1.75 1.75)
+			(drill 1)
+			(layers "*.Cu" "*.Mask")
+			(remove_unused_layers no)
+			(net 3 "unconnected-(J1-Pad3)")
+			(pintype "passive")
+		)
+		(pad "4" thru_hole circle
+			(at 1.7 1.5)
+			(size 1.75 1.75)
+			(drill 1)
+			(layers "*.Cu" "*.Mask")
+			(remove_unused_layers no)
+			(net 1 "unconnected-(J1-Pad4)")
+			(pintype "passive")
+		)
+		(pad "5" thru_hole circle
+			(at -1.7 1.45)
+			(size 1.75 1.75)
+			(drill 1)
+			(layers "*.Cu" "*.Mask")
+			(remove_unused_layers no)
+			(net 6 "unconnected-(J1-Pad5)")
+			(pintype "passive")
+		)
+		(pad "6" thru_hole circle
+			(at -2.25 -0.3)
+			(size 1.75 1.75)
+			(drill 1)
+			(layers "*.Cu" "*.Mask")
+			(remove_unused_layers no)
+			(net 5 "unconnected-(J1-Pad6)")
+			(pintype "passive")
+		)
+	)
